File: src/mx25u1633f-breakout.brd (EAGLE design)
At the start: 18 x 10.6 mm, 4 parts, among them J1 PTH VERT MALE, J2 PTH VERT MALE, U1 MX25U1633F

Commit message: Update CAM files.
Routing:
- net SI: track 9.04 -> 8.28 mm
Changed lines of the file:
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@@
 <setting verticaltext="up"/>
 </settings>
-<grid distance="1" unitdist="mm" unit="mm" style="lines" multiple="1" display="yes" altdistance="0.05" altunitdist="mm" altunit="mm"/>
+<grid distance="0.1" unitdist="mm" unit="mm" style="lines" multiple="1" display="yes" altdistance="0.05" altunitdist="mm" altunit="mm"/>
 <layers>
 <layer number="1" name="Top" color="4" fill="1" visible="yes" active="yes"/>
@@
 </class>
 </classes>
-<designrules name="stella-wearables">
-<description language="en">&lt;b&gt;Stella Wearables Design Rules based on OSH Park Design Rules&lt;/b&gt;
+<designrules name="oshpark-2layer">
+<description language="en">&lt;b&gt;OSH Park Design Rules&lt;/b&gt;
 &lt;p&gt;
 Please make sure your boards conform to these design rules.
@@
 <param name="mtCopper" value="0.035559375mm 0.0356mm 0.0356mm 0.0356mm 0.0356mm 0.0356mm 0.0356mm 0.0356mm 0.0356mm 0.0356mm 0.0356mm 0.0356mm 0.0356mm 0.0356mm 0.0356mm 0.035559375mm"/>
 <param name="mtIsolate" value="1.6mm 0.1499mm 0.2007mm 0.1499mm 0.2007mm 0.1499mm 0.2007mm 0.1499mm 0.2007mm 0.1499mm 0.2007mm 0.1499mm 0.2007mm 0.1499mm 0.2007mm"/>
-<param name="mdWireWire" value="3mil"/>
-<param name="mdWirePad" value="3mil"/>
-<param name="mdWireVia" value="3mil"/>
-<param name="mdPadPad" value="3mil"/>
-<param name="mdPadVia" value="3mil"/>
-<param name="mdViaVia" value="3mil"/>
-<param name="mdSmdPad" value="3mil"/>
-<param name="mdSmdVia" value="3mil"/>
-<param name="mdSmdSmd" value="3mil"/>
+<param name="mdWireWire" value="6mil"/>
+<param name="mdWirePad" value="6mil"/>
+<param name="mdWireVia" value="6mil"/>
+<param name="mdPadPad" value="6mil"/>
+<param name="mdPadVia" value="6mil"/>
+<param name="mdViaVia" value="6mil"/>
+<param name="mdSmdPad" value="6mil"/>
+<param name="mdSmdVia" value="6mil"/>
+<param name="mdSmdSmd" value="6mil"/>
 <param name="mdViaViaSameLayer" value="8mil"/>
 <param name="mnLayersViaInSmd" value="2"/>
@@
 <param name="mdDrill" value="6mil"/>
 <param name="mdSmdStop" value="0mil"/>
-<param name="msWidth" value="3mil"/>
-<param name="msDrill" value="6mil"/>
+<param name="msWidth" value="6mil"/>
+<param name="msDrill" value="10mil"/>
 <param name="msMicroVia" value="10mil"/>
 <param name="msBlindViaRatio" value="0.5"/>
@@
 <contactref element="U1" pad="EP"/>
 <contactref element="C1" pad="2"/>
-<via x="-2.5" y="-0.75" extent="1-16" drill="0.35" diameter="0.1524"/>
+<via x="-2.5" y="-0.85" extent="1-16" drill="0.35" diameter="0.1524"/>
 <via x="0" y="-1.65" extent="1-16" drill="0.35" diameter="0.1524"/>
 <via x="4.5" y="0.8" extent="1-16" drill="0.35" diameter="0.1524"/>
 <wire x1="3.6575" y1="0.8" x2="4.5" y2="0.8" width="0.1524" layer="1"/>
-<wire x1="-1.425" y1="-0.75" x2="-2.5" y2="-0.75" width="0.1524" layer="1"/>
+<wire x1="-1.425" y1="-0.75" x2="-1.825" y2="-0.75" width="0.1524" layer="1"/>
+<wire x1="-1.825" y1="-0.75" x2="-1.925" y2="-0.85" width="0.1524" layer="1"/>
+<wire x1="-1.925" y1="-0.85" x2="-2.5" y2="-0.85" width="0.1524" layer="1"/>
 <contactref element="J1" pad="4"/>
 <wire x1="0" y1="0" x2="0" y2="-1.65" width="0.1524" layer="1"/>
@@
 <signal name="!WP!">
 <contactref element="U1" pad="3"/>
-<wire x1="-1.425" y1="-0.25" x2="-1.85" y2="-0.25" width="0.1524" layer="1"/>
-<wire x1="-2.35" y1="0.25" x2="-1.85" y2="-0.25" width="0.1524" layer="1"/>
 <contactref element="J1" pad="3"/>
-<wire x1="-7.62" y1="-1.27" x2="-6.1" y2="0.25" width="0.1524" layer="1"/>
-<wire x1="-6.1" y1="0.25" x2="-2.35" y2="0.25" width="0.1524" layer="1"/>
+<wire x1="-7.62" y1="-1.27" x2="-6.6" y2="-0.25" width="0.1524" layer="1"/>
+<wire x1="-6.6" y1="-0.25" x2="-1.425" y2="-0.25" width="0.1524" layer="1"/>
 </signal>
 <signal name="!RESET!">
@@
 <signal name="SO">
 <contactref element="U1" pad="2"/>
-<wire x1="-1.425" y1="0.25" x2="-1.85" y2="0.25" width="0.1524" layer="1"/>
-<wire x1="-2.1" y1="0.5" x2="-1.85" y2="0.25" width="0.1524" layer="1"/>
 <contactref element="J1" pad="2"/>
-<wire x1="-7.62" y1="1.27" x2="-6.85" y2="0.5" width="0.1524" layer="1"/>
-<wire x1="-6.85" y1="0.5" x2="-2.1" y2="0.5" width="0.1524" layer="1"/>
+<wire x1="-7.62" y1="1.27" x2="-6.6" y2="0.25" width="0.1524" layer="1"/>
+<wire x1="-6.6" y1="0.25" x2="-1.425" y2="0.25" width="0.1524" layer="1"/>
 </signal>
 <signal name="SI">
 <contactref element="U1" pad="5"/>
-<wire x1="1.425" y1="-0.75" x2="1.85" y2="-0.75" width="0.1524" layer="1"/>
-<wire x1="1.85" y1="-0.75" x2="2.35" y2="-0.25" width="0.1524" layer="1"/>
 <contactref element="J2" pad="4"/>
 <wire x1="6.2" y1="-2.39" x2="7.62" y2="-3.81" width="0.1524" layer="1"/>
-<wire x1="6.05" y1="-0.25" x2="6.2" y2="-0.4" width="0.1524" layer="1"/>
-<wire x1="2.35" y1="-0.25" x2="6.05" y2="-0.25" width="0.1524" layer="1"/>
-<wire x1="6.2" y1="-0.4" x2="6.2" y2="-2.39" width="0.1524" layer="1"/>
+<wire x1="5.95" y1="-0.75" x2="6.2" y2="-1" width="0.1524" layer="1"/>
+<wire x1="1.425" y1="-0.75" x2="5.95" y2="-0.75" width="0.1524" layer="1"/>
+<wire x1="6.2" y1="-1" x2="6.2" y2="-2.39" width="0.1524" layer="1"/>
 </signal>
 <signal name="SCLK">
 <contactref element="U1" pad="6"/>
-<wire x1="1.425" y1="-0.25" x2="1.85" y2="-0.25" width="0.1524" layer="1"/>
-<wire x1="2.1" y1="0" x2="1.85" y2="-0.25" width="0.1524" layer="1"/>
 <contactref element="J2" pad="3"/>
-<wire x1="7.62" y1="-1.27" x2="6.35" y2="0" width="0.1524" layer="1"/>
-<wire x1="6.35" y1="0" x2="2.1" y2="0" width="0.1524" layer="1"/>
+<wire x1="7.62" y1="-1.27" x2="6.6" y2="-0.25" width="0.1524" layer="1"/>
+<wire x1="6.6" y1="-0.25" x2="1.425" y2="-0.25" width="0.1524" layer="1"/>
 </signal>
 <signal name="!CS!">
